File: Eagle Files/Sch1.brd (EAGLE design)
At the start: 62.2 x 53.3 mm, 14 parts

Commit message: Formatting
Parts:
- moved U$1 5.39 mm to (57.1, 41.9)
Changed lines of the file:
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@@
 <wire x1="30.48" y1="40.64" x2="30.48" y2="41.91" width="0.4064" layer="21"/>
 <wire x1="12.7" y1="41.91" x2="12.7" y2="49.53" width="0.4064" layer="21"/>
-<text x="20.32" y="19.05" size="1.778" layer="21">FabCamp 2.0
-2015</text>
-<text x="20.32" y="24.13" size="2.1844" layer="21">UCI</text>
+<text x="21.59" y="19.05" size="1.778" layer="21">FabCamp 2.0
+   2015</text>
+<text x="27.305" y="24.13" size="2.1844" layer="21">UCI</text>
 <hole x="2.54" y="2.54" drill="2.8"/>
 <hole x="59.69" y="2.54" drill="2.8"/>
@@
 <attribute name="VALUE" x="42.164" y="3.429" size="0.8128" layer="21" font="vector" ratio="15"/>
 </element>
-<element name="U$1" library="SparkFun-Aesthetics" package="OSHW-LOGO-L" value="" x="53.34" y="45.72"/>
+<element name="U$1" library="SparkFun-Aesthetics" package="OSHW-LOGO-L" value="" x="57.15" y="41.91"/>
 </elements>
 <signals>
