File: Eagle Files/Sch1.sch (EAGLE design)
At the start: 13 parts

Commit message: Update Files
Parts:
- removed JP1K: M13X22X13, SparkFun-Connectors:M13X22X13
- added C1: (no value), SparkFun-Passives:CAP0805
- added JP1: RASPBERRYPI-B+-GPIO, SparkFun-Boards:RASPBERRYPI-B+-GPIO
- added JP2: (no value), SparkFun-Connectors:M04PTH
- added R5, R6, R7: (no value), SparkFun-Passives:RESISTOR0805-RES
- added SB1, SG1, SR1, SY1: SWITCH-MOMENTARY-2PTH, SparkFun-Electromechanical:SWITCH-MOMENTARY-2PTH
- added SJ1: SOLDERJUMPERNO, SparkFun-Retired:SOLDERJUMPERNO
- added U1: EEPROM-I2CSMD, SparkFun-DigitalIC:EEPROM-I2CSMD
- SB: value blue -> SWITCH-MOMENTARY-2PTH; device adafruit:40-XX -> SparkFun-Electromechanical:SWITCH-MOMENTARY-2PTH
- SG: value green -> SWITCH-MOMENTARY-2PTH; device adafruit:40-XX -> SparkFun-Electromechanical:SWITCH-MOMENTARY-2PTH
- SR: value red -> SWITCH-MOMENTARY-2PTH; device adafruit:40-XX -> SparkFun-Electromechanical:SWITCH-MOMENTARY-2PTH
- SY: value yellow -> SWITCH-MOMENTARY-2PTH; device adafruit:40-XX -> SparkFun-Electromechanical:SWITCH-MOMENTARY-2PTH
Connections:
- new net N$5: JP1.ID_SD, JP2.2, R7.1, U1.SDA
- new net N$6: JP1.ID_SC, JP2.3, R6.1, U1.SCL
- new net N$8: R5.2, SJ1.1, U1.WP
- new net VCC: C1.1, JP1.3.3V@1, JP2.1, R6.2, R7.2, SJ1.2, U1.VCC
- net GND: now also C1.2, JP1.GND@14, JP1.GND@20, JP1.GND@39, JP1.GND@6, JP1.GP13, JP2.4, R5.1, SB.1, SB1.1, SG.1, SG1.1, SR.1, SR1.1, SY.1, SY1.1, U1.A0, U1.A1, U1.A2, U1.VSS; no longer JP1K.6, SB.P, SB.P1, SG.P, SG.P1, SR.P, SR.P1, SY.P, SY.P1
- net LB: now also JP1.GP27; no longer JP1K.13
- net LG: now also JP1.GP17; no longer JP1K.11
- net LR: now also JP1.GP18#; no longer JP1K.15
- net LY: now also JP1.GP22; no longer JP1K.12
- net SB: now also JP1.CE0, SB.2, SB1.2; no longer JP1K.24, SB.S, SB.S1
- net SG: now also JP1.CE1, SG.2, SG1.2; no longer JP1K.26, SG.S, SG.S1
- net SR: now also JP1.GP25, SR.2, SR1.2; no longer JP1K.19, SR.S, SR.S1
- net SY: now also JP1.MOSI, SY.2, SY1.2; no longer JP1K.22, SY.S, SY.S1
Other:
- moved on the sheet: LEDB, LEDG, LEDR, LEDY, R1, R2, R3, R4
